File: kicad/Fidget_Spinner.kicad_pcb (KiCad board)
At the start: 2 copper layers, 81.1 x 74.5 mm, 29 parts, among them Q1 BC846, U1 BAT_HLD_SMD, U2 BAT_HLD_SMD, U3 BAT_HLD_SMD

Commit message: V 10092024
Parts:
- moved U1 0.25 mm to (81.6, 50.3)
- moved U3 0.21 mm to (53.7, 99.4)
Connections:
- U2 pad 1: Net-(U1-Pad2) -> unconnected-(U3-Pad1)
- U2 pad 2: unconnected-(U2-Pad2) -> Net-(Q1-E)
- U3 pad 1: unconnected-(U3-Pad1) -> Net-(U1-Pad2)
- U3 pad 2: Net-(Q1-E) -> unconnected-(U3-Pad1)
Routing:
- net unconnected-(U3-Pad1): track 0.00 -> 56.7 mm
- net Net-(Q1-E): track 48.3 -> 91.6 mm
- net Net-(U1-Pad2): track 86.7 -> 57.5 mm, vias 2 -> 0
- net Net-(S1-E): track 53.6 -> 53.0 mm
- net Net-(D7-A): track 61.7 -> 62.2 mm
Other:
- outline, holes or cut-outs redrawn
- board text added: "B"
- board text added: "C"
- board text added: "E"
- board text added: "G"
- board text added: "S"

Commit message: V 04102024
Other:
- outline, holes or cut-outs redrawn
- board text added: "KHF 10.2024"
- board text removed: "KHF 09.2024"
Changed lines of the file:
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@@
         (effects (font (size 1 1) (thickness 0.15)) (justify mirror))
     )
-    (fp_text value "Micro_Schalter" (at 22.735 6.66) (layer "F.Fab")
+    (fp_text value "Micro_Schalter" (at 5.81 12.25) (layer "F.Fab")
         (effects (font (size 1 1) (thickness 0.15)))
     )
@@
   (gr_line (start 48.9555 59.8346) (end 49.2616 59.4042)
     (stroke (width 0.1) (type solid)) (layer "Edge.Cuts"))
-  (gr_circle (center 69.02 67.53) (end 69.22 67.53)
-    (stroke (width 0.1) (type default)) (fill none) (layer "Edge.Cuts"))
   (gr_line (start 99.6565 80.5045) (end 100.2936 81.0424)
     (stroke (width 0.1) (type solid)) (layer "Edge.Cuts"))
@@
   (gr_line (start 54.8723 112.497) (end 54.1702 112.516)
     (stroke (width 0.1) (type solid)) (layer "Edge.Cuts"))
-  (gr_circle (center 93 69.47) (end 93.2 69.47)
-    (stroke (width 0.1) (type default)) (fill none) (layer "Edge.Cuts"))
   (gr_line (start 42.2024 94.0822) (end 42.4305 93.5987)
     (stroke (width 0.1) (type solid)) (layer "Edge.Cuts"))
-  (gr_circle (center 70.37 69.52) (end 70.57 69.52)
-    (stroke (width 0.1) (type default)) (fill none) (layer "Edge.Cuts"))
   (gr_line (start 69.0201 66.5213) (end 68.9826 67.0729)
     (stroke (width 0.1) (type solid)) (layer "Edge.Cuts"))
@@
   (gr_line (start 80.6742 98.4276) (end 79.6446 98.5447)
     (stroke (width 0.1) (type solid)) (layer "Edge.Cuts"))
-  (gr_circle (center 70.71 67.9) (end 70.91 67.9)
-    (stroke (width 0.1) (type default)) (fill none) (layer "Edge.Cuts"))
   (gr_line (start 41.2211 101.4109) (end 41.1378 100.7553)
     (stroke (width 0.1) (type solid)) (layer "Edge.Cuts"))
@@
   (gr_line (start 95.0297 62.1926) (end 95.2262 61.694)
     (stroke (width 0.1) (type solid)) (layer "Edge.Cuts"))
-  (gr_circle (center 92.6 67.93) (end 92.8 67.93)
-    (stroke (width 0.1) (type default)) (fill none) (layer "Edge.Cuts"))
   (gr_line (start 92.1221 62.4202) (end 92.0964 63.0704)
     (stroke (width 0.1) (type solid)) (layer "Edge.Cuts"))
@@
   (gr_line (start 101.5667 55.6555) (end 102.0768 55.4829)
     (stroke (width 0.1) (type solid)) (layer "Edge.Cuts"))
-  (gr_circle (center 94.38 67.52) (end 94.58 67.52)
-    (stroke (width 0.1) (type default)) (fill none) (layer "Edge.Cuts"))
   (gr_line (start 112.324 74.4379) (end 111.9093 74.7638)
     (stroke (width 0.1) (type solid)) (layer "Edge.Cuts"))
@@
   (gr_line (start 55.0244 85.807) (end 55.6313 85.5906)
     (stroke (width 0.1) (type solid)) (layer "Edge.Cuts"))
-  (gr_circle (center 68.68 69.15) (end 68.88 69.15)
-    (stroke (width 0.1) (type default)) (fill none) (layer "Edge.Cuts"))
   (gr_line (start 68.4223 69.5959) (end 68.2752 70.0012)
     (stroke (width 0.1) (type solid)) (layer "Edge.Cuts"))
@@
   (gr_line (start 102.5977 55.335) (end 103.1288 55.2124)
     (stroke (width 0.1) (type solid)) (layer "Edge.Cuts"))
-  (gr_circle (center 94.78 69.06) (end 94.98 69.06)
-    (stroke (width 0.1) (type default)) (fill none) (layer "Edge.Cuts"))
   (gr_line (start 99.9569 75.5731) (end 99.5961 75.3636)
     (stroke (width 0.1) (type solid)) (layer "Edge.Cuts"))
@@
   (gr_line (start 53.2991 56.0772) (end 53.7854 55.8573)
     (stroke (width 0.1) (type solid)) (layer "Edge.Cuts"))
-  (gr_text "KHF 09.2024 " (at 86.52 96.84) (layer "B.Cu")
+  (gr_text "KHF 10.2024 " (at 86.52 96.84) (layer "B.Cu")
     (effects (font (size 1 1) (thickness 0.15)) (justify left bottom mirror))
   )
@@
     (effects (font (size 1 1) (thickness 0.15)))
   )
-  (gr_text "KHF 09.2024" (at 86.52 96.86) (layer "B.Mask")
+  (gr_text "KHF 10.2024" (at 86.52 96.86) (layer "B.Mask")
     (effects (font (size 1 1) (thickness 0.15)) (justify left bottom mirror))
   )
